File: Ports.sch (KiCad schematic (older format))
At the start: 12 parts, among them J1 SIO, J5 Joystick_Port, J6 Joystick_Port, J8 Keyboard

Commit message: Tracking
Parts:
- C93, C94, C95: footprint Atari:C_Axial_L5.1mm_D2.5mm_P12.50mm_Horizontal -> Capacitor_SMD:C_1206_3216Metric_Pad1.42x1.75mm_HandSolder
- R95: footprint Atari:R_Axial_DIN0207_L3.6mm_D2.2mm_P10.16mm_Horizontal -> Resistor_SMD:R_1206_3216Metric_Pad1.42x1.75mm_HandSolder
Changed lines of the file:
@@
 F 0 "R95" V 4550 3075 50  0000 C CNN
 F 1 "1k" V 4500 2925 50  0000 C CNN
-F 2 "Atari:R_Axial_DIN0207_L3.6mm_D2.2mm_P10.16mm_Horizontal" V 4480 3075 50  0001 C CNN
+F 2 "Resistor_SMD:R_1206_3216Metric_Pad1.42x1.75mm_HandSolder" V 4480 3075 50  0001 C CNN
 F 3 "~" H 4550 3075 50  0001 C CNN
 	1    4550 3075
@@
 F 0 "C93" H 3700 3300 50  0000 L CNN
 F 1 "100nF" H 3700 3150 50  0000 L CNN
-F 2 "Atari:C_Axial_L5.1mm_D2.5mm_P12.50mm_Horizontal" H 3713 3075 50  0001 C CNN
+F 2 "Capacitor_SMD:C_1206_3216Metric_Pad1.42x1.75mm_HandSolder" H 3713 3075 50  0001 C CNN
 F 3 "~" H 3675 3225 50  0001 C CNN
 	1    3675 3225
@@
 F 0 "C95" H 4900 3300 50  0000 L CNN
 F 1 "10nF" H 4850 3150 50  0000 L CNN
-F 2 "Atari:C_Axial_L5.1mm_D2.5mm_P12.50mm_Horizontal" H 5088 3075 50  0001 C CNN
+F 2 "Capacitor_SMD:C_1206_3216Metric_Pad1.42x1.75mm_HandSolder" H 5088 3075 50  0001 C CNN
 F 3 "~" H 5050 3225 50  0001 C CNN
 	1    5050 3225
@@
 F 0 "C94" H 4000 3300 50  0000 L CNN
 F 1 "10nF" H 3950 3150 50  0000 L CNN
-F 2 "Atari:C_Axial_L5.1mm_D2.5mm_P12.50mm_Horizontal" H 4188 3075 50  0001 C CNN
+F 2 "Capacitor_SMD:C_1206_3216Metric_Pad1.42x1.75mm_HandSolder" H 4188 3075 50  0001 C CNN
 F 3 "~" H 4150 3225 50  0001 C CNN
 	1    4150 3225

Commit message: Change THT on SMD
Parts:
- C102: footprint Atari:C_Axial_L5.1mm_D2.5mm_P12.50mm_Horizontal -> Capacitor_SMD:C_1206_3216Metric_Pad1.42x1.75mm_HandSolder
- FB102, FB12, L25: footprint Atari:L_Axial_L7.0mm_D3.3mm_P12.50mm_Horizontal_Fastron_MICC -> Inductor_SMD:L_1812_4532Metric_Pad1.30x3.40mm_HandSolder
Changed lines of the file:
@@
 F 0 "FB102" V 8000 2500 50  0000 C CNN
 F 1 "Ferrite_Bead" V 8350 2500 50  0000 C CNN
-F 2 "Atari:L_Axial_L7.0mm_D3.3mm_P12.50mm_Horizontal_Fastron_MICC" V 8105 2525 50  0001 C CNN
+F 2 "Inductor_SMD:L_1812_4532Metric_Pad1.30x3.40mm_HandSolder" V 8105 2525 50  0001 C CNN
 F 3 "~" H 8175 2525 50  0001 C CNN
 	1    8175 2525
@@
 F 0 "C102" H 8740 2896 50  0000 L CNN
 F 1 "1nF" H 8740 2805 50  0000 L CNN
-F 2 "Atari:C_Axial_L5.1mm_D2.5mm_P12.50mm_Horizontal" H 8663 2700 50  0001 C CNN
+F 2 "Capacitor_SMD:C_1206_3216Metric_Pad1.42x1.75mm_HandSolder" H 8663 2700 50  0001 C CNN
 F 3 "~" H 8625 2850 50  0001 C CNN
 	1    8625 2850
@@
 F 0 "FB12" H 7275 2175 50  0000 R CNN
 F 1 "Ferrite_Bead" V 6875 2225 50  0000 R CNN
-F 2 "Atari:L_Axial_L7.0mm_D3.3mm_P12.50mm_Horizontal_Fastron_MICC" V 6980 2325 50  0001 C CNN
+F 2 "Inductor_SMD:L_1812_4532Metric_Pad1.30x3.40mm_HandSolder" V 6980 2325 50  0001 C CNN
 F 3 "~" H 7050 2325 50  0001 C CNN
 	1    7050 2325
@@
 F 0 "L25" V 7369 2525 50  0000 C CNN
 F 1 "10uH" V 7460 2525 50  0000 C CNN
-F 2 "Atari:L_Axial_L7.0mm_D3.3mm_P12.50mm_Horizontal_Fastron_MICC" H 7550 2525 50  0001 C CNN
+F 2 "Inductor_SMD:L_1812_4532Metric_Pad1.30x3.40mm_HandSolder" H 7550 2525 50  0001 C CNN
 F 3 "~" H 7550 2525 50  0001 C CNN
 	1    7550 2525
