File: Sally_Antic.sch (KiCad schematic (older format))
At the start: 10 parts, among them U18 74LS08, U7 Antic, U8 Sally

Commit message: OSS and Basic in PLCC
Parts:
- R33: footprint Atari:R_Axial_DIN0207_L3.6mm_D2.2mm_P10.16mm_Horizontal -> Resistor_SMD:R_1206_3216Metric_Pad1.42x1.75mm_HandSolder
Changed lines of the file:
@@
 F 0 "R33" H 2295 1571 50  0000 L CNN
 F 1 "3k" H 2295 1480 50  0000 L CNN
-F 2 "Atari:R_Axial_DIN0207_L3.6mm_D2.2mm_P10.16mm_Horizontal" V 2155 1525 50  0001 C CNN
+F 2 "Resistor_SMD:R_1206_3216Metric_Pad1.42x1.75mm_HandSolder" V 2155 1525 50  0001 C CNN
 F 3 "~" H 2225 1525 50  0001 C CNN
 	1    2225 1525
