File: Atari 130XE 1MB.kicad_pcb (KiCad board)
At the start: 2 copper layers, 324 x 204 mm, 349 parts, among them J1 SIO, J10 Mem_on_off, J100 cond, J101 cond, J102 pin, J103 pin, J104 pin, J105 pin, J106 pin, J107 pin, J108 pin, J109 pin, J110 pin, J111 pin, J2 Video, J201 Diagnostic, J202 Diag, J210 Diag, J211 Diag, J212 Diag, J24 Cartridge, J4 Expansion, J5 Joystick_Port, J6 Joystick_Port, J7 Power, J8 Keyboard, M1 Modulator, Q1 2N3904, Q2 2N3904, Q3 2N3904, Q4 2N3906, Q6 2N3904, SW1 Switch_power_on, U1 LM358, U10 DRAM_4464, U17 GTIA, U18 74LS08, U19 LM555, U2 74LS138, U20 4050, U21 74LS74, U22 POKEY, U23 PIA, U24 CD4051B, U25 CD4051B, U3 MMU, U4 BASIC_ROM, U40 GAL20V8_DIP, U41 74LS157, U42 74LS175, U43 DRAM_1MB_4bit, U44 DRAM_1MB_4bit, U5 27C128, U6 Freddie, U7 Antic, U8 Sally, U9 DRAM_4464, Y1 Crystal, Y2 4,43 MHz

Commit message: Simm finished
Parts:
- moved C123 87.3 mm to (86.9, 144.1), turned to 180 degrees
Routing:
- net +5VA: track 1890.8 -> 1975.7 mm
- net RAS: track 112.6 -> 185.7 mm, vias 3 -> 6
- net GND: track 1557.7 -> 1606.5 mm, vias 8 -> 30
- net Net-(U41-Pad4): track 17.5 -> 64.6 mm, vias 0 -> 2
- net Net-(U41-Pad7): track 18.6 -> 62.6 mm, vias 2 -> 4
- net Net-(R111-Pad1): track 21.1 -> 61.1 mm
- net PB7: track 311.7 -> 309.2 mm
- net DQ5: track 59.8 -> 62.2 mm
- net PB1: track 307.8 -> 305.6 mm
- net PB6: track 305.1 -> 303.5 mm
- net DQ3: track 87.7 -> 89.2 mm
- net RA0: track 113.3 -> 114.6 mm
- net RA7: track 154.0 -> 155.3 mm
- net RA1: track 114.0 -> 114.9 mm
- net FA14: track 32.4 -> 31.5 mm
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
Commit message: Tracking
Parts:
- C69, C70, C93, C94, C95: footprint Atari:C_Axial_L5.1mm_D2.5mm_P12.50mm_Horizontal -> Capacitor_SMD:C_1206_3216Metric_Pad1.42x1.75mm_HandSolder
- R134, R135, R136, R137, R138, R139, R140, R141, R142, R143, R144, R145, R146, R147, R148, R149, R150, R151, R152, R153, R89, R90, R95: footprint Atari:R_Axial_DIN0207_L3.6mm_D2.2mm_P10.16mm_Horizontal -> Resistor_SMD:R_1206_3216Metric_Pad1.42x1.75mm_HandSolder
- moved R142 44.1 mm to (294.5, 202.8), turned to 90 degrees
- moved R140 40.6 mm to (297.1, 202.8), turned to 90 degrees
- moved R138 37.0 mm to (299.6, 202.8), turned to 90 degrees
- moved R134 32.9 mm to (335.2, 202.8), turned to 90 degrees
- moved R137 32.4 mm to (332.6, 202.8), turned to 90 degrees
- moved R135 30.8 mm to (337.7, 202.8), turned to 90 degrees
- moved U24 29.7 mm to (304.8, 194.5)
- moved R136 29.0 mm to (340.2, 202.8), turned to 90 degrees
- moved R150 29.0 mm to (330.1, 202.8), turned to 90 degrees
- moved C69 28.8 mm to (305.7, 183.8)
- moved R89 27.3 mm to (285.9, 200.0)
- moved R139 25.4 mm to (312.3, 202.8), turned to 90 degrees
- moved R152 24.5 mm to (292.0, 202.8), turned to 90 degrees
- moved R146 24.4 mm to (325.0, 202.8), turned to 90 degrees
- moved R144 21.8 mm to (314.9, 202.8), turned to 90 degrees
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Routing:
- net IN4: track 59.3 -> 4.58 mm, vias 1 -> 0
- net OUT3: track 58.1 -> 4.57 mm
- net OUT5: track 53.7 -> 4.57 mm
- net IN0: track 52.1 -> 4.57 mm, vias 1 -> 0
- net BSC: track 51.2 -> 4.57 mm
- net Net-(R140-Pad2): track 58.4 -> 12.9 mm
- net OUT7: track 49.3 -> 4.57 mm
- net Net-(R138-Pad2): track 64.9 -> 20.4 mm, vias 1 -> 0
- net IN3: track 47.3 -> 4.58 mm, vias 1 -> 0
- net +5VA: track 1975.7 -> 2016.4 mm
- net START: track 43.6 -> 4.58 mm
- net IN6: track 42.7 -> 4.57 mm, vias 1 -> 0
- net SELECT: track 41.4 -> 4.58 mm
- net OPTION: track 38.6 -> 4.58 mm
- net OUT6: track 34.7 -> 4.57 mm
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
Commit message: Change THT on SMD
Parts:
- C102, C200, C201, C85, C86, C87, C88, C89, C90, C91, C92: footprint Atari:C_Axial_L5.1mm_D2.5mm_P12.50mm_Horizontal -> Capacitor_SMD:C_1206_3216Metric_Pad1.42x1.75mm_HandSolder
- C98: footprint Capacitor_THT:CP_Axial_L11.0mm_D6.0mm_P18.00mm_Horizontal -> Capacitor_THT:CP_Radial_D5.0mm_P2.00mm
- D5: footprint Diode_THT:D_DO-35_SOD27_P12.70mm_Horizontal -> Diode_SMD:D_1206_3216Metric_Pad1.42x1.75mm_HandSolder
- FB102, FB12, L14, L19, L20, L21, L22, L25, L26, L27, L28, L29: footprint Atari:L_Axial_L7.0mm_D3.3mm_P12.50mm_Horizontal_Fastron_MICC -> Inductor_SMD:L_1812_4532Metric_Pad1.30x3.40mm_HandSolder
- R120, R121, R122, R123, R124, R125, R126, R127, R200, R206, R39, R40, R96: footprint Atari:R_Axial_DIN0207_L3.6mm_D2.2mm_P10.16mm_Horizontal -> Resistor_SMD:R_1206_3216Metric_Pad1.42x1.75mm_HandSolder
- moved R206 220.5 mm to (86.5, 174.3), turned to 270 degrees
- moved C200 106.0 mm to (345.6, 189.4)
- moved R200 94.2 mm to (345.6, 186.8), turned to 0 degrees
- moved U19 93.7 mm to (333.6, 194.5)
- moved R39 92.2 mm to (345.6, 194.6), turned to 0 degrees
- moved R40 87.9 mm to (345.6, 192.0), turned to 180 degrees
- moved C201 79.5 mm to (330.6, 187.8), turned to 270 degrees
- moved C92 50.6 mm to (305.5, 126.1)
- moved C91 43.1 mm to (305.5, 121.5)
- moved C88 40.5 mm to (314.3, 126.1)
- moved C90 35.6 mm to (305.5, 116.8)
- moved C89 28.1 mm to (305.5, 112.2)
- moved D5 26.1 mm to (289.8, 174.8), turned to 90 degrees
- moved C87 26.1 mm to (314.3, 121.5), turned to 180 degrees
- moved L22 23.9 mm to (304.9, 106.6), turned to 0 degrees
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Connections:
- J212 pad 12: BO2 -> D7XX
- J212 pad 7: D7XX -> BO2
Routing:
- net +5VA: track 2016.4 -> 1898.0 mm, vias 27 -> 28
- net GND: track 1593.2 -> 1514.2 mm
- net Net-(L14-Pad1): track 81.6 -> 9.90 mm, vias 2 -> 0
- net Net-(R89-Pad1): track 30.5 -> 91.3 mm, vias 0 -> 2
- net Net-(D5-Pad2): track 22.3 -> 72.4 mm, vias 0 -> 1
- net Net-(R134-Pad2): track 120.1 -> 165.0 mm
- net Net-(R135-Pad2): track 122.2 -> 165.9 mm
- net Net-(R136-Pad2): track 124.2 -> 167.0 mm
- net Net-(C89-Pad1): track 39.8 -> 5.66 mm
- net PB5: track 262.0 -> 231.1 mm
- net FWD1: track 53.7 -> 81.4 mm, vias 0 -> 1
- net Net-(C90-Pad1): track 42.3 -> 18.4 mm
- net BACK1: track 59.2 -> 82.1 mm, vias 0 -> 1
- net Net-(C86-Pad1): track 39.1 -> 16.3 mm
- net Net-(C85-Pad1): track 28.6 -> 5.81 mm
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
Commit message: OSS and Basic in PLCC
Parts:
- removed J108, J109, J110, J111: pin, Connector_PinHeader_2.00mm:PinHeader_1x01_P2.00mm_Vertical
- removed J211: Diag, Connector_PinHeader_2.54mm:PinHeader_1x01_P2.54mm_Vertical
- removed J212: Diag, Connector_PinHeader_2.54mm:PinHeader_2x06_P2.54mm_Vertical
- C27, C28, C62, C63, C64, C65, C66, C68, C71, C72, C73, C74, C75, C76, C77, C78: footprint Atari:C_Axial_L5.1mm_D2.5mm_P12.50mm_Horizontal -> Capacitor_SMD:C_1206_3216Metric_Pad1.42x1.75mm_HandSolder
- L15, L16, L17, L18: footprint Atari:L_Axial_L7.0mm_D3.3mm_P12.50mm_Horizontal_Fastron_MICC -> Inductor_SMD:L_1812_4532Metric_Pad1.30x3.40mm_HandSolder
- R128, R129, R130, R131, R19, R23, R24, R25, R33, R501, R76, R77, R78, R79, R80, R81, R82, R83, R84, R85, R86, R87, R88: footprint Atari:R_Axial_DIN0207_L3.6mm_D2.2mm_P10.16mm_Horizontal -> Resistor_SMD:R_1206_3216Metric_Pad1.42x1.75mm_HandSolder
- U4: value BASIC_ROM -> 27C010; footprint Package_DIP:DIP-24_W15.24mm_Socket -> Atari:PLCC-32_THT-Socket
- U5: value 27C128 -> 27C010; footprint Package_DIP:DIP-28_W15.24mm_Socket -> Atari:PLCC-32_THT-Socket
- moved R87 204.0 mm to (103.1, 186.0), turned to 0 degrees
- moved R88 194.5 mm to (103.1, 197.7), turned to 0 degrees
- moved R85 187.1 mm to (103.1, 183.7), turned to 0 degrees
- moved R80 134.6 mm to (123.4, 160.1), turned to 180 degrees
- moved C73 69.7 mm to (335.8, 144.5), turned to 0 degrees
- moved L15 59.5 mm to (336.5, 141.4)
- moved C74 55.7 mm to (335.9, 133.6), turned to 0 degrees
- moved C27 49.2 mm to (247.6, 191.5)
- moved C28 49.1 mm to (247.6, 188.0)
- moved C62 44.7 mm to (306.5, 169.3), turned to 270 degrees
- moved L16 44.6 mm to (336.6, 130.4)
- moved C102 40.7 mm to (344.4, 129.7)
- moved FB102 40.6 mm to (345.1, 132.9)
- moved L25 40.4 mm to (345.1, 136.9), turned to 0 degrees
- moved FB12 37.0 mm to (345.1, 140.8), turned to 180 degrees
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Connections:
- U2 pad 7: D7XX -> (no net)
- U2 pad 9: D6XX -> (no net)
- U3 pad 13: BASIC -> (no net)
- U4 pad 1: A7 -> +5VA
- U4 pad 10: D1 -> A2
- U4 pad 11: D2 -> A1
- U4 pad 12: GND -> A0
- U4 pad 13: D3 -> D0
- U4 pad 14: D4 -> D1
- U4 pad 15: D5 -> D2
- U4 pad 16: D6 -> GND
- U4 pad 17: D7 -> D3
- U4 pad 18: A11 -> D4
- U4 pad 19: A10 -> D5
- U4 pad 2: A6 -> (no net)
- U4 pad 20: BASIC -> D6
- U4 pad 21: A12 -> D7
- U4 pad 22: A9 -> (no net)
- U4 pad 23: A8 -> A10
- U4 pad 24: +5VA -> (no net)
- U4 pad 3: A5 -> (no net)
- U4 pad 4: A4 -> A12
- U4 pad 5: A3 -> A7
- U4 pad 6: A2 -> A6
- U4 pad 7: A1 -> A5
- U4 pad 8: A0 -> A4
- U4 pad 9: D0 -> A3
- U5 pad 10: A0 -> A2
- U5 pad 11: D0 -> A1
- U5 pad 12: D1 -> A0
- U5 pad 13: D2 -> D0
- U5 pad 14: GND -> D1
- U5 pad 15: D3 -> D2
- U5 pad 16: D4 -> GND
- U5 pad 17: D5 -> D3
- U5 pad 18: D6 -> D4
- U5 pad 19: D7 -> D5
- U5 pad 2: A12 -> Net-(U5-Pad2)
- U5 pad 20: OS -> D6
- U5 pad 21: A10 -> D7
- U5 pad 22: OS -> Net-(U5-Pad22)
- U5 pad 23: A11 -> A10
- U5 pad 24: A9 -> Net-(U5-Pad24)
- U5 pad 25: A8 -> A11
- U5 pad 26: A13 -> A9
- U5 pad 27: +5VA -> A8
- U5 pad 28: +5VA -> A13
- U5 pad 3: A7 -> Net-(U5-Pad3)
- U5 pad 4: A6 -> A12
- U5 pad 5: A5 -> A7
- U5 pad 6: A4 -> A6
- U5 pad 7: A3 -> A5
- U5 pad 8: A2 -> A4
- U5 pad 9: A1 -> A3
Routing:
- net (no net): track 0.00 -> 290.6 mm, vias 0 -> 7
- net D6XX: track 163.8 -> 0.00 mm, vias 3 -> 0
- net D7XX: track 119.2 -> 0.00 mm, vias 3 -> 0
- net GND: track 1514.2 -> 1397.5 mm, vias 28 -> 33
- net BASIC: track 88.1 -> 0.00 mm, vias 1 -> 0
- net A9: track 338.3 -> 253.4 mm, vias 5 -> 3
- net A8: track 344.7 -> 262.1 mm, vias 5 -> 3
- net Net-(C74-Pad1): track 81.1 -> 10.1 mm
- net Net-(C73-Pad1): track 80.9 -> 10.0 mm
- net PB1: track 305.6 -> 243.9 mm, vias 8 -> 6
- net O2: track 454.4 -> 394.2 mm, vias 6 -> 5
- net POT_B1: track 38.7 -> 95.9 mm, vias 0 -> 1
- net PB6: track 303.5 -> 247.0 mm, vias 5 -> 4
- net A11: track 345.6 -> 290.9 mm, vias 4 -> 2
- net +5VA: track 1898.0 -> 1952.5 mm, vias 28 -> 31
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Other:
- board text removed: "BO2"
- board text removed: "CCTL"
- board text removed: "D6XX"
- board text removed: "D7XX"
- board text removed: "MPD"
- board text removed: "RD4"
- board text removed: "RD5"
- board text removed: "RST"
- board text removed: "S4"
- board text removed: "S5"

Commit message: SuperCart
Parts:
- added C207: 100nF, Capacitor_SMD:C_1206_3216Metric_Pad1.42x1.75mm_HandSolder, F.Cu at (258.8, 216.6)
- added J211: Conn_01x02, Connector_PinHeader_2.54mm:PinHeader_1x02_P2.54mm_Vertical, F.Cu at (258.2, 210.0)
- added R502: 1k, Resistor_SMD:R_1206_3216Metric_Pad1.42x1.75mm_HandSolder, F.Cu at (263.5, 209.4)
- added R503: 10k, Resistor_SMD:R_1206_3216Metric_Pad1.42x1.75mm_HandSolder, F.Cu at (263.5, 212.7)
- added U100: 74LS157, Package_SO:SOIC-16_3.9x9.9mm_P1.27mm, F.Cu at (251.6, 213.5)
- moved C28 53.8 mm to (195.0, 199.5), turned to 180 degrees
- moved C27 32.5 mm to (225.7, 215.5), turned to 180 degrees
Connections:
- U3 pad 13: (no net) -> BASIC
- U3 pad 15: OS -> (no net)
- U4 pad 22: (no net) -> Net-(U100-Pad9)
- U4 pad 24: (no net) -> Net-(U100-Pad9)
- U4 pad 28: (no net) -> Net-(U100-Pad7)
- U4 pad 4: A12 -> Net-(U100-Pad4)
- U5 pad 2: Net-(U5-Pad2) -> (no net)
- U5 pad 22: Net-(U5-Pad22) -> (no net)
- U5 pad 24: Net-(U5-Pad24) -> (no net)
- U5 pad 29: Net-(U5-Pad29) -> (no net)
- U5 pad 3: Net-(U5-Pad3) -> (no net)
Routing:
- net (no net): track 290.6 -> 139.1 mm, vias 7 -> 3
- net D1: track 515.4 -> 605.0 mm, vias 5 -> 10
- net D2: track 532.8 -> 607.1 mm, vias 6 -> 10
- net D0: track 514.0 -> 587.4 mm, vias 6 -> 10
- net A10: track 261.9 -> 334.8 mm, vias 3 -> 7
- net A9: track 253.4 -> 325.7 mm, vias 3 -> 5
- net A11: track 290.9 -> 360.8 mm, vias 2 -> 5
- net O2: track 394.2 -> 458.7 mm, vias 5 -> 6
- net D3: track 442.4 -> 505.8 mm, vias 5 -> 6
- net BASIC: track 0.00 -> 60.5 mm, vias 0 -> 1
- net PB0: track 209.9 -> 270.2 mm, vias 6 -> 7
- net A8: track 262.1 -> 321.0 mm, vias 3 -> 5
- net PB4: track 204.7 -> 262.7 mm, vias 2 -> 3
- net PB6: track 247.0 -> 305.0 mm, vias 4 -> 5
- net PB3: track 202.8 -> 260.5 mm, vias 2 -> 3
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