File: Audio and Video.sch (KiCad schematic (older format))
At the start: 32 parts, among them J106 pin, J107 pin, M1 Modulator, U1 LM358, U19 LM555

Commit message: Change THT on SMD
Parts:
- C200, C201: footprint Atari:C_Axial_L5.1mm_D2.5mm_P12.50mm_Horizontal -> Capacitor_SMD:C_1206_3216Metric_Pad1.42x1.75mm_HandSolder
- L14: footprint Atari:L_Axial_L7.0mm_D3.3mm_P12.50mm_Horizontal_Fastron_MICC -> Inductor_SMD:L_1812_4532Metric_Pad1.30x3.40mm_HandSolder
- R200, R39, R40: footprint Atari:R_Axial_DIN0207_L3.6mm_D2.2mm_P10.16mm_Horizontal -> Resistor_SMD:R_1206_3216Metric_Pad1.42x1.75mm_HandSolder
Changed lines of the file:
@@
 F 0 "C201" H 9865 4371 50  0000 L CNN
 F 1 "100nF" H 9865 4280 50  0000 L CNN
-F 2 "Atari:C_Axial_L5.1mm_D2.5mm_P12.50mm_Horizontal" H 9788 4175 50  0001 C CNN
+F 2 "Capacitor_SMD:C_1206_3216Metric_Pad1.42x1.75mm_HandSolder" H 9788 4175 50  0001 C CNN
 F 3 "~" H 9750 4325 50  0001 C CNN
 	1    9750 4325
@@
 F 0 "R200" V 7550 4425 50  0000 L CNN
 F 1 "470k" V 7650 4425 50  0000 L CNN
-F 2 "Atari:R_Axial_DIN0207_L3.6mm_D2.2mm_P10.16mm_Horizontal" V 7480 4525 50  0001 C CNN
+F 2 "Resistor_SMD:R_1206_3216Metric_Pad1.42x1.75mm_HandSolder" V 7480 4525 50  0001 C CNN
 F 3 "~" H 7550 4525 50  0001 C CNN
 	1    7550 4525
@@
 F 0 "C200" V 6998 4250 50  0000 C CNN
 F 1 "100nF" V 7089 4250 50  0000 C CNN
-F 2 "Atari:C_Axial_L5.1mm_D2.5mm_P12.50mm_Horizontal" H 7288 4100 50  0001 C CNN
+F 2 "Capacitor_SMD:C_1206_3216Metric_Pad1.42x1.75mm_HandSolder" H 7288 4100 50  0001 C CNN
 F 3 "~" H 7250 4250 50  0001 C CNN
 	1    7250 4250
@@
 F 0 "R39" H 6700 4025 50  0000 L CNN
 F 1 "56k" H 6700 3925 50  0000 L CNN
-F 2 "Atari:R_Axial_DIN0207_L3.6mm_D2.2mm_P10.16mm_Horizontal" V 6830 3925 50  0001 C CNN
+F 2 "Resistor_SMD:R_1206_3216Metric_Pad1.42x1.75mm_HandSolder" V 6830 3925 50  0001 C CNN
 F 3 "~" H 6900 3925 50  0001 C CNN
 	1    6900 3925
@@
 F 0 "R40" H 6700 4675 50  0000 L CNN
 F 1 "100" H 6700 4600 50  0000 L CNN
-F 2 "Atari:R_Axial_DIN0207_L3.6mm_D2.2mm_P10.16mm_Horizontal" V 6830 4525 50  0001 C CNN
+F 2 "Resistor_SMD:R_1206_3216Metric_Pad1.42x1.75mm_HandSolder" V 6830 4525 50  0001 C CNN
 F 3 "~" H 6900 4525 50  0001 C CNN
 	1    6900 4525
@@
 F 0 "L14" V 6394 4800 50  0000 C CNN
 F 1 "22uH" V 6485 4800 50  0000 C CNN
-F 2 "Atari:L_Axial_L7.0mm_D3.3mm_P12.50mm_Horizontal_Fastron_MICC" H 6575 4800 50  0001 C CNN
+F 2 "Inductor_SMD:L_1812_4532Metric_Pad1.30x3.40mm_HandSolder" H 6575 4800 50  0001 C CNN
 F 3 "~" H 6575 4800 50  0001 C CNN
 	1    6575 4800

Commit message: Final modification
Parts:
- added C160: 1n, Capacitor_SMD:C_1206_3216Metric_Pad1.42x1.75mm_HandSolder, symbol Device:C
- added J22: C, Connector_PinHeader_2.54mm:PinHeader_1x01_P2.54mm_Vertical, symbol Connector_Generic:Conn_01x01
- added Q10, Q11: PN2222A, Package_TO_SOT_THT:TO-92_Inline, symbol Transistor_BJT:PN2222A
- added R160: 33, Resistor_SMD:R_1206_3216Metric_Pad1.42x1.75mm_HandSolder, symbol Device:R
- added R161: 18, Resistor_SMD:R_1206_3216Metric_Pad1.42x1.75mm_HandSolder, symbol Device:R
- added R162: 82, Resistor_SMD:R_1206_3216Metric_Pad1.42x1.75mm_HandSolder, symbol Device:R
- added R163: 180, Resistor_SMD:R_1206_3216Metric_Pad1.42x1.75mm_HandSolder, symbol Device:R
- C19, C20, C22: footprint Capacitor_THT:CP_Radial_D8.0mm_P3.50mm -> Capacitor_THT:C_Rect_L7.2mm_W7.2mm_P5.00mm_FKS2_FKP2_MKS2_MKP2
- C24: footprint Capacitor_THT:CP_Axial_L11.0mm_D6.0mm_P18.00mm_Horizontal -> Capacitor_THT:CP_Radial_D7.5mm_P2.50mm
Connections:
- net +5VA: now also Q10.3 (C), Q11.3 (C)
- net COLOR: now also Q11.2 (B)
- net GND: now also J22.1 (Pin_1), R162.2, R163.2
- net MONO_MOD: now also Q10.2 (B)
- net COMPOSITE_A: now reaches FB7.1, M1.1 (Composite)
- net COMPOSITE_A: now also R161.2, R162.1
- new net: Q10.1 (E), R160.1
- new net: C160.1, R160.2, R161.1
- new net: C160.2, Q11.1 (E), R163.1
Changed lines of the file:
@@
 F 0 "C20" V 3325 2725 50  0000 L CNN
 F 1 "4,7uF" V 3625 2725 50  0000 L CNN
-F 2 "Capacitor_THT:CP_Radial_D8.0mm_P3.50mm" H 3513 2650 50  0001 C CNN
+F 2 "Capacitor_THT:C_Rect_L7.2mm_W7.2mm_P5.00mm_FKS2_FKP2_MKS2_MKP2" H 3513 2650 50  0001 C CNN
 F 3 "~" H 3475 2800 50  0001 C CNN
 	1    3475 2800
@@
 F 0 "C19" H 3300 2250 50  0000 L CNN
 F 1 "4,7uF" H 3050 2250 50  0000 L CNN
-F 2 "Capacitor_THT:CP_Radial_D8.0mm_P3.50mm" H 3313 2200 50  0001 C CNN
+F 2 "Capacitor_THT:C_Rect_L7.2mm_W7.2mm_P5.00mm_FKS2_FKP2_MKS2_MKP2" H 3313 2200 50  0001 C CNN
 F 3 "~" H 3275 2350 50  0001 C CNN
 	1    3275 2350
@@
 F 0 "C24" H 4418 3271 50  0000 L CNN
 F 1 "10uF" H 4418 3180 50  0000 L CNN
-F 2 "Capacitor_THT:CP_Axial_L11.0mm_D6.0mm_P18.00mm_Horizontal" H 4338 3075 50  0001 C CNN
+F 2 "Capacitor_THT:CP_Radial_D7.5mm_P2.50mm" H 4338 3075 50  0001 C CNN
 F 3 "~" H 4300 3225 50  0001 C CNN
 	1    4300 3225
@@
 	4100 1875 4100 2100
 Connection ~ 4100 2100
-$Comp
-L Device:C C23
-U 1 1 603243E3
-P 3625 1400
-F 0 "C23" V 3500 1200 50  0000 L CNN
-F 1 "47nF" V 3550 1475 50  0000 L CNN
-F 2 "Atari:C_Axial_L5.1mm_D2.5mm_P12.50mm_Horizontal" H 3663 1250 50  0001 C CNN
-F 3 "~" H 3625 1400 50  0001 C CNN
-	1    3625 1400
-	0    1    1    0
-$EndComp
 Wire Wire Line
 	4100 1575 4100 1400
@@
 $EndComp
 Wire Wire Line
-	7250 1500 7825 1500
+	7250 1500 7500 1500
 Text GLabel 875  1625 0    50   Input ~ 0
 EXTAUDIO
-$Comp
-L Device:C C22
-U 1 1 6039DB1C
-P 1275 1625
-F 0 "C22" V 1400 1575 50  0000 L CNN
-F 1 "4,7uF" V 1200 1350 50  0000 L CNN
-F 2 "Capacitor_THT:CP_Radial_D8.0mm_P3.50mm" H 1313 1475 50  0001 C CNN
-F 3 "~" H 1275 1625 50  0001 C CNN
-	1    1275 1625
-	0    -1   -1   0
-$EndComp
 Wire Wire Line
 	875  1625 1125 1625
@@
 Wire Wire Line
 	1200 3350 1600 3350
+$Comp
+L Device:C C22
+U 1 1 6039DB1C
+P 1275 1625
+F 0 "C22" V 1400 1575 50  0000 L CNN
+F 1 "4,7uF" V 1200 1350 50  0000 L CNN
+F 2 "Capacitor_THT:C_Rect_L7.2mm_W7.2mm_P5.00mm_FKS2_FKP2_MKS2_MKP2" H 1313 1475 50  0001 C CNN
+F 3 "~" H 1275 1625 50  0001 C CNN
+	1    1275 1625
+	0    -1   -1   0
+$EndComp
+$Comp
+L Device:C C23
+U 1 1 603243E3
+P 3625 1400
+F 0 "C23" V 3500 1200 50  0000 L CNN
+F 1 "47nF" V 3550 1475 50  0000 L CNN
+F 2 "Atari:C_Axial_L5.1mm_D2.5mm_P12.50mm_Horizontal" H 3663 1250 50  0001 C CNN
+F 3 "~" H 3625 1400 50  0001 C CNN
+	1    3625 1400
+	0    1    1    0
+$EndComp
+$Comp
+L Connector_Generic:Conn_01x01 J22
+U 1 1 60DE4CF7
+P 5475 3275
+F 0 "J22" V 5439 3187 50  0000 R CNN
+F 1 "C" V 5348 3187 50  0000 R CNN
+F 2 "Connector_PinHeader_2.54mm:PinHeader_1x01_P2.54mm_Vertical" H 5475 3275 50  0001 C CNN
+F 3 "~" H 5475 3275 50  0001 C CNN
+	1    5475 3275
+	0    -1   -1   0
+$EndComp
+$Comp
+L power:GND #PWR0293
+U 1 1 60DF1471
+P 5475 3575
+F 0 "#PWR0293" H 5475 3325 50  0001 C CNN
+F 1 "GND" H 5480 3402 50  0000 C CNN
+F 2 "" H 5475 3575 50  0001 C CNN
+F 3 "" H 5475 3575 50  0001 C CNN
+	1    5475 3575
+	1    0    0    -1
+$EndComp
+Wire Wire Line
+	5475 3475 5475 3575
+Text GLabel 4025 5025 0    50   Input ~ 0
+MONO_MOD
+$Comp
+L Transistor_BJT:PN2222A Q10
+U 1 1 60DCB735
+P 4400 5025
+F 0 "Q10" H 4590 5071 50  0000 L CNN
+F 1 "PN2222A" H 4590 4980 50  0000 L CNN
+F 2 "Package_TO_SOT_THT:TO-92_Inline" H 4600 4950 50  0001 L CIN
+F 3 "http://www.fairchildsemi.com/ds/PN/PN2222A.pdf" H 4400 5025 50  0001 L CNN
+	1    4400 5025
+	1    0    0    -1
+$EndComp
+Wire Wire Line
+	4025 5025 4200 5025
+$Comp
+L power:+5VA #PWR0294
+U 1 1 60DCF214
+P 4500 4525
+F 0 "#PWR0294" H 4500 4375 50  0001 C CNN
+F 1 "+5VA" H 4515 4698 50  0000 C CNN
+F 2 "" H 4500 4525 50  0001 C CNN
+F 3 "" H 4500 4525 50  0001 C CNN
+	1    4500 4525
+	1    0    0    -1
+$EndComp
+Wire Wire Line
+	4500 4825 4500 4525
+$Comp
+L Device:R R160
+U 1 1 60DD68AD
+P 4500 5550
+F 0 "R160" H 4570 5596 50  0000 L CNN
+F 1 "33" H 4570 5505 50  0000 L CNN
+F 2 "Resistor_SMD:R_1206_3216Metric_Pad1.42x1.75mm_HandSolder" V 4430 5550 50  0001 C CNN
+F 3 "~" H 4500 5550 50  0001 C CNN
+	1    4500 5550
+	1    0    0    -1
+$EndComp
+Wire Wire Line
+	4500 5225 4500 5400
+$Comp
+L Device:R R161
+U 1 1 60DD9BE3
+P 4500 6000
+F 0 "R161" H 4570 6046 50  0000 L CNN
+F 1 "18" H 4570 5955 50  0000 L CNN
+F 2 "Resistor_SMD:R_1206_3216Metric_Pad1.42x1.75mm_HandSolder" V 4430 6000 50  0001 C CNN
+F 3 "~" H 4500 6000 50  0001 C CNN
+	1    4500 6000
+	1    0    0    -1
+$EndComp
+Wire Wire Line
+	4500 5700 4500 5800
+$Comp
+L Device:R R162
+U 1 1 60DDD184
+P 4500 6475
+F 0 "R162" H 4570 6521 50  0000 L CNN
+F 1 "82" H 4570 6430 50  0000 L CNN
+F 2 "Resistor_SMD:R_1206_3216Metric_Pad1.42x1.75mm_HandSolder" V 4430 6475 50  0001 C CNN
+F 3 "~" H 4500 6475 50  0001 C CNN
+	1    4500 6475
+	1    0    0    -1
+$EndComp
+Wire Wire Line
+	4500 6150 4500 6250
+$Comp
+L power:GND #PWR0295
+U 1 1 60DE0647
+P 4500 6800
+F 0 "#PWR0295" H 4500 6550 50  0001 C CNN
+F 1 "GND" H 4505 6627 50  0000 C CNN
+F 2 "" H 4500 6800 50  0001 C CNN
+F 3 "" H 4500 6800 50  0001 C CNN
+	1    4500 6800
+	1    0    0    -1
+$EndComp
+Wire Wire Line
+	4500 6625 4500 6800
+$Comp
+L Device:C C160
+U 1 1 60DEA334
+P 3950 5800
+F 0 "C160" V 3698 5800 50  0000 C CNN
+F 1 "1n" V 3789 5800 50  0000 C CNN
+F 2 "Capacitor_SMD:C_1206_3216Metric_Pad1.42x1.75mm_HandSolder" H 3988 5650 50  0001 C CNN
+F 3 "~" H 3950 5800 50  0001 C CNN
+	1    3950 5800
+	0    1    1    0
+$EndComp
+Wire Wire Line
+	4100 5800 4500 5800
+Connection ~ 4500 5800
+Wire Wire Line
+	4500 5800 4500 5850
+$Comp
+L Transistor_BJT:PN2222A Q11
+U 1 1 60DEE4F4
+P 2975 5400
+F 0 "Q11" H 3165 5446 50  0000 L CNN
+F 1 "PN2222A" H 3165 5355 50  0000 L CNN
+F 2 "Package_TO_SOT_THT:TO-92_Inline" H 3175 5325 50  0001 L CIN
+F 3 "http://www.fairchildsemi.com/ds/PN/PN2222A.pdf" H 2975 5400 50  0001 L CNN
+	1    2975 5400
+	1    0    0    -1
+$EndComp
+Wire Wire Line
+	3075 5600 3075 5800
+Wire Wire Line
+	3075 5800 3800 5800
+$Comp
+L Device:R R163
+U 1 1 60DF21C4
+P 3075 6450
+F 0 "R163" H 3145 6496 50  0000 L CNN
+F 1 "180" H 3145 6405 50  0000 L CNN
+F 2 "Resistor_SMD:R_1206_3216Metric_Pad1.42x1.75mm_HandSolder" V 3005 6450 50  0001 C CNN
+F 3 "~" H 3075 6450 50  0001 C CNN
+	1    3075 6450
+	1    0    0    -1
+$EndComp
+Wire Wire Line
+	3075 5800 3075 6300
+Connection ~ 3075 5800
+$Comp
+L power:GND #PWR0296
+U 1 1 60DF6C36
+P 3075 6825
+F 0 "#PWR0296" H 3075 6575 50  0001 C CNN
+F 1 "GND" H 3080 6652 50  0000 C CNN
+F 2 "" H 3075 6825 50  0001 C CNN
+F 3 "" H 3075 6825 50  0001 C CNN
+	1    3075 6825
+	1    0    0    -1
+$EndComp
+Wire Wire Line
+	3075 6600 3075 6825
+$Comp
+L power:+5VA #PWR0297
+U 1 1 60DFBFA9
+P 3075 4525
+F 0 "#PWR0297" H 3075 4375 50  0001 C CNN
+F 1 "+5VA" H 3090 4698 50  0000 C CNN
+F 2 "" H 3075 4525 50  0001 C CNN
+F 3 "" H 3075 4525 50  0001 C CNN
+	1    3075 4525
+	1    0    0    -1
+$EndComp
+Wire Wire Line
+	3075 4525 3075 5200
+Text GLabel 2425 5400 0    50   Input ~ 0
+COLOR
+Wire Wire Line
+	2425 5400 2775 5400
+Wire Wire Line
+	4925 6250 4500 6250
+Connection ~ 4500 6250
+Wire Wire Line
+	4500 6250 4500 6325
+Text GLabel 7500 1250 1    50   Input ~ 0
+COMPOSITE_A
+Wire Wire Line
+	7500 1250 7500 1500
+Connection ~ 7500 1500
+Wire Wire Line
+	7500 1500 7825 1500
+Text GLabel 4925 6250 2    50   Input ~ 0
+COMPOSITE_A
 $EndSCHEMATC
