File: Freddie.sch (KiCad schematic (older format))
At the start: 16 parts, among them J100 cond, J101 cond, J200 Diag, U18 74LS08, U6 Freddie, Y1 Crystal

Commit message: SIMM update
Parts:
- removed J200: Diag, Connector_PinHeader_2.54mm:PinHeader_1x12_P2.54mm_Vertical, symbol Connector_Generic:Conn_01x12
Connections:
- net labels removed: HALT, REF
- wire segments 35 -> 34
Changed lines of the file:
@@
 EESchema Schematic File Version 4
-LIBS:Atari 130XE-cache
+LIBS:Atari 130XE 1MB-cache
 EELAYER 29 0
 EELAYER END
 $Descr A4 11693 8268
 encoding utf-8
-Sheet 5 15
+Sheet 5 16
 Title ""
 Date ""
@@
 	10900 3225 10900 2850
 Connection ~ 10275 3225
-Text GLabel 7950 4325 0    50   Input ~ 0
-CAS
-Text GLabel 7950 4425 0    50   Input ~ 0
-WRT
-Text GLabel 7950 4525 0    50   Input ~ 0
-RAS
-Text GLabel 7950 4025 0    50   Input ~ 0
-RW
-Text GLabel 7950 4125 0    50   Input ~ 0
-OSC
-Text GLabel 7950 3725 0    50   Input ~ 0
-O2
-Text GLabel 7950 4225 0    50   Input ~ 0
-CASINH
-Text GLabel 7950 3925 0    50   Input ~ 0
-EXTSEL
-Text GLabel 7950 3825 0    50   Input ~ 0
-REF
-Text GLabel 7950 4825 0    50   Input ~ 0
-GND
-$Comp
-L Connector_Generic:Conn_01x12 J200
-U 1 1 6047EC37
-P 8150 4225
-F 0 "J200" H 8230 4217 50  0000 L CNN
-F 1 "Diag" H 8230 4126 50  0000 L CNN
-F 2 "Connector_PinHeader_2.54mm:PinHeader_1x12_P2.54mm_Vertical" H 8150 4225 50  0001 C CNN
-F 3 "~" H 8150 4225 50  0001 C CNN
-	1    8150 4225
-	1    0    0    -1
-$EndComp
-Text GLabel 7950 4625 0    50   Input ~ 0
-HALT
-Wire Wire Line
-	7950 4725 7950 4825
 $EndSCHEMATC

Commit message: OSS and Basic in PLCC
Parts:
- R19: footprint Atari:R_Axial_DIN0207_L3.6mm_D2.2mm_P10.16mm_Horizontal -> Resistor_SMD:R_1206_3216Metric_Pad1.42x1.75mm_HandSolder
Changed lines of the file:
@@
 F 0 "R19" V 8350 2900 50  0000 C CNN
 F 1 "3k" V 8425 2900 50  0000 C CNN
-F 2 "Atari:R_Axial_DIN0207_L3.6mm_D2.2mm_P10.16mm_Horizontal" V 8280 2900 50  0001 C CNN
+F 2 "Resistor_SMD:R_1206_3216Metric_Pad1.42x1.75mm_HandSolder" V 8280 2900 50  0001 C CNN
 F 3 "~" H 8350 2900 50  0001 C CNN
 	1    8350 2900

Commit message: Final modification
Parts:
- added J50: Test_signal, Connector_PinHeader_2.54mm:PinHeader_2x05_P2.54mm_Vertical, symbol Connector_Generic:Conn_02x05_Odd_Even
- added J51: To_GND, Connector_PinHeader_2.54mm:PinHeader_1x02_P2.54mm_Vertical, symbol Connector_Generic:Conn_01x02
Connections:
- net CAS: now also J50.5 (Pin_5)
- net CASINH: now also J50.2 (Pin_2)
- net FA14: now also J50.9 (Pin_9)
- net FA15: now also J50.7 (Pin_7)
- net GND: now also J51.1 (Pin_1), J51.2 (Pin_2)
- net O2: now also J50.8 (Pin_8)
- net OSC: now also J50.4 (Pin_4)
- net RAS: now also J50.3 (Pin_3)
- net RW: now also J50.6 (Pin_6)
- net WRT: now also J50.1 (Pin_1)
- new net REF: J50.10 (Pin_10)
Changed lines of the file:
@@
 	10900 3225 10900 2850
 Connection ~ 10275 3225
+$Comp
+L Connector_Generic:Conn_02x05_Odd_Even J50
+U 1 1 60E3B546
+P 2525 4350
+F 0 "J50" H 2575 4767 50  0000 C CNN
+F 1 "Test_signal" H 2575 4676 50  0000 C CNN
+F 2 "Connector_PinHeader_2.54mm:PinHeader_2x05_P2.54mm_Vertical" H 2525 4350 50  0001 C CNN
+F 3 "~" H 2525 4350 50  0001 C CNN
+	1    2525 4350
+	1    0    0    -1
+$EndComp
+Text GLabel 2825 4550 2    50   Input ~ 0
+REF
+Text GLabel 2825 4450 2    50   Input ~ 0
+O2
+Text GLabel 2825 4350 2    50   Input ~ 0
+RW
+Text GLabel 2825 4250 2    50   Input ~ 0
+OSC
+Text GLabel 2825 4150 2    50   Input ~ 0
+CASINH
+Text GLabel 2325 4150 0    50   Input ~ 0
+WRT
+Text GLabel 2325 4250 0    50   Input ~ 0
+RAS
+Text GLabel 2325 4350 0    50   Input ~ 0
+CAS
+Text GLabel 2325 4450 0    50   Input ~ 0
+FA15
+Text GLabel 2325 4550 0    50   Input ~ 0
+FA14
+$Comp
+L Connector_Generic:Conn_01x02 J51
+U 1 1 60E51996
+P 3800 4325
+F 0 "J51" H 3880 4317 50  0000 L CNN
+F 1 "To_GND" H 3880 4226 50  0000 L CNN
+F 2 "Connector_PinHeader_2.54mm:PinHeader_1x02_P2.54mm_Vertical" H 3800 4325 50  0001 C CNN
+F 3 "~" H 3800 4325 50  0001 C CNN
+	1    3800 4325
+	1    0    0    -1
+$EndComp
+Wire Wire Line
+	3600 4325 3600 4425
+$Comp
+L power:GND #PWR0298
+U 1 1 60E5426E
+P 3600 4575
+F 0 "#PWR0298" H 3600 4325 50  0001 C CNN
+F 1 "GND" H 3605 4402 50  0000 C CNN
+F 2 "" H 3600 4575 50  0001 C CNN
+F 3 "" H 3600 4575 50  0001 C CNN
+	1    3600 4575
+	1    0    0    -1
+$EndComp
+Wire Wire Line
+	3600 4425 3600 4575
+Connection ~ 3600 4425
 $EndSCHEMATC
