File: GTIA.sch (KiCad schematic (older format))
At the start: 78 parts, among them J102 pin, J103 pin, J104 pin, J105 pin, J2 Video, J202 Diag, J210 Diag, Q1 2N3904, Q2 2N3904, Q3 2N3904, Q6 2N3904, U17 GTIA, U18 74LS08, U20 4050, U21 74LS74, Y2 4,43 MHz

Commit message: Tracking
Parts:
- R134, R135, R136: footprint Atari:R_Axial_DIN0207_L3.6mm_D2.2mm_P10.16mm_Horizontal -> Resistor_SMD:R_1206_3216Metric_Pad1.42x1.75mm_HandSolder
Changed lines of the file:
@@
 F 0 "R134" V 4725 2975 50  0000 C CNN
 F 1 "470" V 4675 3150 50  0000 C CNN
-F 2 "Atari:R_Axial_DIN0207_L3.6mm_D2.2mm_P10.16mm_Horizontal" V 4655 2975 50  0001 C CNN
+F 2 "Resistor_SMD:R_1206_3216Metric_Pad1.42x1.75mm_HandSolder" V 4655 2975 50  0001 C CNN
 F 3 "~" H 4725 2975 50  0001 C CNN
 	1    4725 2975
@@
 F 0 "R135" V 4725 3075 50  0000 C CNN
 F 1 "470" V 4675 3250 50  0000 C CNN
-F 2 "Atari:R_Axial_DIN0207_L3.6mm_D2.2mm_P10.16mm_Horizontal" V 4655 3075 50  0001 C CNN
+F 2 "Resistor_SMD:R_1206_3216Metric_Pad1.42x1.75mm_HandSolder" V 4655 3075 50  0001 C CNN
 F 3 "~" H 4725 3075 50  0001 C CNN
 	1    4725 3075
@@
 F 0 "R136" V 4725 3175 50  0000 C CNN
 F 1 "470" V 4675 3350 50  0000 C CNN
-F 2 "Atari:R_Axial_DIN0207_L3.6mm_D2.2mm_P10.16mm_Horizontal" V 4655 3175 50  0001 C CNN
+F 2 "Resistor_SMD:R_1206_3216Metric_Pad1.42x1.75mm_HandSolder" V 4655 3175 50  0001 C CNN
 F 3 "~" H 4725 3175 50  0001 C CNN
 	1    4725 3175

Commit message: Final modification
Parts:
- C96, C97: footprint Atari:C_Axial_L5.1mm_D2.5mm_P12.50mm_Horizontal -> Capacitor_SMD:C_1206_3216Metric_Pad1.42x1.75mm_HandSolder
- L23, L30: footprint Atari:L_Axial_L7.0mm_D3.3mm_P12.50mm_Horizontal_Fastron_MICC -> Inductor_SMD:L_1812_4532Metric_Pad1.30x3.40mm_HandSolder
- R132, R133: footprint Atari:R_Axial_DIN0207_L3.6mm_D2.2mm_P10.16mm_Horizontal -> Resistor_SMD:R_1206_3216Metric_Pad1.42x1.75mm_HandSolder
Changed lines of the file:
@@
 F 0 "R132" V 4875 3325 50  0000 C CNN
 F 1 "220" V 4825 3500 50  0000 C CNN
-F 2 "Atari:R_Axial_DIN0207_L3.6mm_D2.2mm_P10.16mm_Horizontal" V 4805 3325 50  0001 C CNN
+F 2 "Resistor_SMD:R_1206_3216Metric_Pad1.42x1.75mm_HandSolder" V 4805 3325 50  0001 C CNN
 F 3 "~" H 4875 3325 50  0001 C CNN
 	1    4875 3325
@@
 F 0 "R133" V 4875 3425 50  0000 C CNN
 F 1 "220" V 4825 3600 50  0000 C CNN
-F 2 "Atari:R_Axial_DIN0207_L3.6mm_D2.2mm_P10.16mm_Horizontal" V 4805 3425 50  0001 C CNN
+F 2 "Resistor_SMD:R_1206_3216Metric_Pad1.42x1.75mm_HandSolder" V 4805 3425 50  0001 C CNN
 F 3 "~" H 4875 3425 50  0001 C CNN
 	1    4875 3425
@@
 F 0 "L30" V 5625 3325 50  0000 C CNN
 F 1 "100uH" V 5625 3575 50  0000 C CNN
-F 2 "Atari:L_Axial_L7.0mm_D3.3mm_P12.50mm_Horizontal_Fastron_MICC" H 5675 3325 50  0001 C CNN
+F 2 "Inductor_SMD:L_1812_4532Metric_Pad1.30x3.40mm_HandSolder" H 5675 3325 50  0001 C CNN
 F 3 "~" H 5675 3325 50  0001 C CNN
 	1    5675 3325
@@
 F 0 "L23" V 5750 3425 50  0000 C CNN
 F 1 "100uH" V 5750 3675 50  0000 C CNN
-F 2 "Atari:L_Axial_L7.0mm_D3.3mm_P12.50mm_Horizontal_Fastron_MICC" H 5675 3425 50  0001 C CNN
+F 2 "Inductor_SMD:L_1812_4532Metric_Pad1.30x3.40mm_HandSolder" H 5675 3425 50  0001 C CNN
 F 3 "~" H 5675 3425 50  0001 C CNN
 	1    5675 3425
@@
 F 0 "C97" H 5250 3550 50  0000 C CNN
 F 1 "1nF" H 5225 3725 50  0000 C CNN
-F 2 "Atari:C_Axial_L5.1mm_D2.5mm_P12.50mm_Horizontal" H 5188 3475 50  0001 C CNN
+F 2 "Capacitor_SMD:C_1206_3216Metric_Pad1.42x1.75mm_HandSolder" H 5188 3475 50  0001 C CNN
 F 3 "~" H 5150 3625 50  0001 C CNN
 	1    5150 3625
@@
 F 0 "C96" H 5550 3550 50  0000 C CNN
 F 1 "1nF" H 5525 3725 50  0000 C CNN
-F 2 "Atari:C_Axial_L5.1mm_D2.5mm_P12.50mm_Horizontal" H 5488 3475 50  0001 C CNN
+F 2 "Capacitor_SMD:C_1206_3216Metric_Pad1.42x1.75mm_HandSolder" H 5488 3475 50  0001 C CNN
 F 3 "~" H 5450 3625 50  0001 C CNN
 	1    5450 3625
