File: Memory.sch (KiCad schematic (older format))
At the start: 22 parts, among them U10 DRAM_4464, U11 DRAM_4464, U12 DRAM_4464, U34 MMMU_GAL, U35 74LS95, U9 DRAM_4464

Commit message: SIMM update
Parts:
- removed C101, C103: 100nF, Atari:C_Axial_L5.1mm_D2.5mm_P12.50mm_Horizontal, symbol Device:C
- removed C34, C35: 100nF, Capacitor_THT:C_Axial_L3.8mm_D2.6mm_P7.50mm_Horizontal, symbol Device:C
- removed R110, R111: 33, Atari:R_Axial_DIN0207_L3.6mm_D2.2mm_P10.16mm_Horizontal, symbol Device:R
- removed U11, U12: DRAM_4464, Package_DIP:DIP-18_W7.62mm, symbol Atari:DRAM_4464
- removed U34: MMMU_GAL, Package_DIP:DIP-20_W7.62mm_Socket, symbol Atari:MMMU_GAL
- removed U35: 74LS95, Package_DIP:DIP-14_W7.62mm_Socket, symbol 74xx:74LS95
Connections:
- net labels removed: A14, A15, CAS, CASBNK, FA14, FA15, HALT, O2, PB2, PB3, PB4, PB5
- wire segments 88 -> 20
- no-connect marks 4 -> 0
Other:
- moved on the sheet: C36, C37, R207, R208, R209, R210, R211, R212, R213, R214, U10, U9

Commit message: Final modification
Parts:
- added R100, R101, R102, R103, R104, R105, R106, R107: 10k, Atari:R_Axial_DIN0207_L3.6mm_D2.2mm_P10.16mm_Horizontal, symbol Device:R
Connections:
- net +5VA: now also R100.2, R101.2, R102.2, R103.2, R104.2, R105.2, R106.2, R107.2
- net DQ0: now also R105.1
- net DQ1: now also R103.1
- net DQ2: now also R104.1
- net DQ3: now also R102.1
- net DQ4: now also R100.1
- net DQ5: now also R101.1
- net DQ6: now also R106.1
- net DQ7: now also R107.1
Changed lines of the file:
@@
 Wire Wire Line
 	7125 4825 5675 4825
+$Comp
+L Device:R R100
+U 1 1 60D91D41
+P 2925 3775
+F 0 "R100" V 2925 3775 50  0000 C CNN
+F 1 "10k" V 2875 3600 50  0000 C CNN
+F 2 "Atari:R_Axial_DIN0207_L3.6mm_D2.2mm_P10.16mm_Horizontal" V 2855 3775 50  0001 C CNN
+F 3 "~" H 2925 3775 50  0001 C CNN
+	1    2925 3775
+	0    1    1    0
+$EndComp
+Text GLabel 3075 3775 2    50   Input ~ 0
+DQ4
+$Comp
+L power:+5VA #PWR0286
+U 1 1 60D9284E
+P 2425 3500
+F 0 "#PWR0286" H 2425 3350 50  0001 C CNN
+F 1 "+5VA" H 2440 3673 50  0000 C CNN
+F 2 "" H 2425 3500 50  0001 C CNN
+F 3 "" H 2425 3500 50  0001 C CNN
+	1    2425 3500
+	1    0    0    -1
+$EndComp
+Wire Wire Line
+	2775 3775 2425 3775
+Wire Wire Line
+	2425 3775 2425 3500
+$Comp
+L Device:R R101
+U 1 1 60D9A894
+P 2925 3900
+F 0 "R101" V 2925 3900 50  0000 C CNN
+F 1 "10k" V 2875 3725 50  0000 C CNN
+F 2 "Atari:R_Axial_DIN0207_L3.6mm_D2.2mm_P10.16mm_Horizontal" V 2855 3900 50  0001 C CNN
+F 3 "~" H 2925 3900 50  0001 C CNN
+	1    2925 3900
+	0    1    1    0
+$EndComp
+Text GLabel 3075 3900 2    50   Input ~ 0
+DQ5
+Wire Wire Line
+	2775 3900 2425 3900
+Wire Wire Line
+	2425 3900 2425 3775
+Connection ~ 2425 3775
+$Comp
+L Device:R R102
+U 1 1 60D9DE57
+P 2925 4025
+F 0 "R102" V 2925 4025 50  0000 C CNN
+F 1 "10k" V 2875 3850 50  0000 C CNN
+F 2 "Atari:R_Axial_DIN0207_L3.6mm_D2.2mm_P10.16mm_Horizontal" V 2855 4025 50  0001 C CNN
+F 3 "~" H 2925 4025 50  0001 C CNN
+	1    2925 4025
+	0    1    1    0
+$EndComp
+Text GLabel 3075 4025 2    50   Input ~ 0
+DQ3
+Wire Wire Line
+	2775 4025 2425 4025
+Wire Wire Line
+	2425 4025 2425 3900
+Connection ~ 2425 3900
+$Comp
+L Device:R R103
+U 1 1 60D8E68E
+P 2925 4150
+F 0 "R103" V 2925 4150 50  0000 C CNN
+F 1 "10k" V 2875 3975 50  0000 C CNN
+F 2 "Atari:R_Axial_DIN0207_L3.6mm_D2.2mm_P10.16mm_Horizontal" V 2855 4150 50  0001 C CNN
+F 3 "~" H 2925 4150 50  0001 C CNN
+	1    2925 4150
+	0    1    1    0
+$EndComp
+Text GLabel 3075 4150 2    50   Input ~ 0
+DQ1
+Wire Wire Line
+	2775 4150 2425 4150
+Wire Wire Line
+	2425 4150 2425 4025
+Connection ~ 2425 4025
+$Comp
+L Device:R R104
+U 1 1 60D8F264
+P 2925 4275
+F 0 "R104" V 2925 4275 50  0000 C CNN
+F 1 "10k" V 2875 4100 50  0000 C CNN
+F 2 "Atari:R_Axial_DIN0207_L3.6mm_D2.2mm_P10.16mm_Horizontal" V 2855 4275 50  0001 C CNN
+F 3 "~" H 2925 4275 50  0001 C CNN
+	1    2925 4275
+	0    1    1    0
+$EndComp
+Text GLabel 3075 4275 2    50   Input ~ 0
+DQ2
+Wire Wire Line
+	2425 4150 2425 4275
+Wire Wire Line
+	2425 4275 2775 4275
+Connection ~ 2425 4150
+$Comp
+L Device:R R105
+U 1 1 60D9380E
+P 2925 4400
+F 0 "R105" V 2925 4400 50  0000 C CNN
+F 1 "10k" V 2875 4225 50  0000 C CNN
+F 2 "Atari:R_Axial_DIN0207_L3.6mm_D2.2mm_P10.16mm_Horizontal" V 2855 4400 50  0001 C CNN
+F 3 "~" H 2925 4400 50  0001 C CNN
+	1    2925 4400
+	0    1    1    0
+$EndComp
+Text GLabel 3075 4400 2    50   Input ~ 0
+DQ0
+Wire Wire Line
+	2425 4275 2425 4400
+Wire Wire Line
+	2425 4400 2775 4400
+Connection ~ 2425 4275
+$Comp
+L Device:R R106
+U 1 1 60D96A99
+P 2925 4525
+F 0 "R106" V 2925 4525 50  0000 C CNN
+F 1 "10k" V 2875 4350 50  0000 C CNN
+F 2 "Atari:R_Axial_DIN0207_L3.6mm_D2.2mm_P10.16mm_Horizontal" V 2855 4525 50  0001 C CNN
+F 3 "~" H 2925 4525 50  0001 C CNN
+	1    2925 4525
+	0    1    1    0
+$EndComp
+Text GLabel 3075 4525 2    50   Input ~ 0
+DQ6
+$Comp
+L Device:R R107
+U 1 1 60D96E46
+P 2925 4650
+F 0 "R107" V 2925 4650 50  0000 C CNN
+F 1 "10k" V 2875 4475 50  0000 C CNN
+F 2 "Atari:R_Axial_DIN0207_L3.6mm_D2.2mm_P10.16mm_Horizontal" V 2855 4650 50  0001 C CNN
+F 3 "~" H 2925 4650 50  0001 C CNN
+	1    2925 4650
+	0    1    1    0
+$EndComp
+Text GLabel 3075 4650 2    50   Input ~ 0
+DQ7
+Wire Wire Line
+	2775 4525 2425 4525
+Wire Wire Line
+	2425 4525 2425 4400
+Connection ~ 2425 4400
+Wire Wire Line
+	2775 4650 2425 4650
+Wire Wire Line
+	2425 4650 2425 4525
+Connection ~ 2425 4525
 $EndSCHEMATC
