File: PIA.sch (KiCad schematic (older format))
At the start: 51 parts, among them Q4 2N3906, U23 PIA

Commit message: Change THT on SMD
Parts:
- C85, C86, C87, C88, C89, C90, C91, C92: footprint Atari:C_Axial_L5.1mm_D2.5mm_P12.50mm_Horizontal -> Capacitor_SMD:C_1206_3216Metric_Pad1.42x1.75mm_HandSolder
- L19, L20, L21, L22, L26, L27, L28, L29: footprint Atari:L_Axial_L7.0mm_D3.3mm_P12.50mm_Horizontal_Fastron_MICC -> Inductor_SMD:L_1812_4532Metric_Pad1.30x3.40mm_HandSolder
- R120, R121, R122, R123, R124, R125, R126, R127, R206: footprint Atari:R_Axial_DIN0207_L3.6mm_D2.2mm_P10.16mm_Horizontal -> Resistor_SMD:R_1206_3216Metric_Pad1.42x1.75mm_HandSolder
Changed lines of the file:
@@
 F 0 "R206" V 2600 2325 50  0000 L CNN
 F 1 "3k3" H 2500 2575 50  0000 L CNN
-F 2 "Atari:R_Axial_DIN0207_L3.6mm_D2.2mm_P10.16mm_Horizontal" V 2530 2425 50  0001 C CNN
+F 2 "Resistor_SMD:R_1206_3216Metric_Pad1.42x1.75mm_HandSolder" V 2530 2425 50  0001 C CNN
 F 3 "~" H 2600 2425 50  0001 C CNN
 	1    2600 2425
@@
 F 0 "R120" V 4775 3675 50  0000 L CNN
 F 1 "220" V 4725 3900 50  0000 L CNN
-F 2 "Atari:R_Axial_DIN0207_L3.6mm_D2.2mm_P10.16mm_Horizontal" V 4705 3775 50  0001 C CNN
+F 2 "Resistor_SMD:R_1206_3216Metric_Pad1.42x1.75mm_HandSolder" V 4705 3775 50  0001 C CNN
 F 3 "~" H 4775 3775 50  0001 C CNN
 	1    4775 3775
@@
 F 0 "R121" V 4775 3775 50  0000 L CNN
 F 1 "220" V 4725 4000 50  0000 L CNN
-F 2 "Atari:R_Axial_DIN0207_L3.6mm_D2.2mm_P10.16mm_Horizontal" V 4705 3875 50  0001 C CNN
+F 2 "Resistor_SMD:R_1206_3216Metric_Pad1.42x1.75mm_HandSolder" V 4705 3875 50  0001 C CNN
 F 3 "~" H 4775 3875 50  0001 C CNN
 	1    4775 3875
@@
 F 0 "R122" V 4775 3875 50  0000 L CNN
 F 1 "220" V 4725 4100 50  0000 L CNN
-F 2 "Atari:R_Axial_DIN0207_L3.6mm_D2.2mm_P10.16mm_Horizontal" V 4705 3975 50  0001 C CNN
+F 2 "Resistor_SMD:R_1206_3216Metric_Pad1.42x1.75mm_HandSolder" V 4705 3975 50  0001 C CNN
 F 3 "~" H 4775 3975 50  0001 C CNN
 	1    4775 3975
@@
 F 0 "R123" V 4775 3975 50  0000 L CNN
 F 1 "220" V 4725 4200 50  0000 L CNN
-F 2 "Atari:R_Axial_DIN0207_L3.6mm_D2.2mm_P10.16mm_Horizontal" V 4705 4075 50  0001 C CNN
+F 2 "Resistor_SMD:R_1206_3216Metric_Pad1.42x1.75mm_HandSolder" V 4705 4075 50  0001 C CNN
 F 3 "~" H 4775 4075 50  0001 C CNN
 	1    4775 4075
@@
 F 0 "R124" V 4775 4075 50  0000 L CNN
 F 1 "220" V 4725 4300 50  0000 L CNN
-F 2 "Atari:R_Axial_DIN0207_L3.6mm_D2.2mm_P10.16mm_Horizontal" V 4705 4175 50  0001 C CNN
+F 2 "Resistor_SMD:R_1206_3216Metric_Pad1.42x1.75mm_HandSolder" V 4705 4175 50  0001 C CNN
 F 3 "~" H 4775 4175 50  0001 C CNN
 	1    4775 4175
@@
 F 0 "R125" V 4775 4175 50  0000 L CNN
 F 1 "220" V 4725 4400 50  0000 L CNN
-F 2 "Atari:R_Axial_DIN0207_L3.6mm_D2.2mm_P10.16mm_Horizontal" V 4705 4275 50  0001 C CNN
+F 2 "Resistor_SMD:R_1206_3216Metric_Pad1.42x1.75mm_HandSolder" V 4705 4275 50  0001 C CNN
 F 3 "~" H 4775 4275 50  0001 C CNN
 	1    4775 4275
@@
 F 0 "R126" V 4775 4275 50  0000 L CNN
 F 1 "220" V 4725 4500 50  0000 L CNN
-F 2 "Atari:R_Axial_DIN0207_L3.6mm_D2.2mm_P10.16mm_Horizontal" V 4705 4375 50  0001 C CNN
+F 2 "Resistor_SMD:R_1206_3216Metric_Pad1.42x1.75mm_HandSolder" V 4705 4375 50  0001 C CNN
 F 3 "~" H 4775 4375 50  0001 C CNN
 	1    4775 4375
@@
 F 0 "R127" V 4775 4375 50  0000 L CNN
 F 1 "220" V 4725 4600 50  0000 L CNN
-F 2 "Atari:R_Axial_DIN0207_L3.6mm_D2.2mm_P10.16mm_Horizontal" V 4705 4475 50  0001 C CNN
+F 2 "Resistor_SMD:R_1206_3216Metric_Pad1.42x1.75mm_HandSolder" V 4705 4475 50  0001 C CNN
 F 3 "~" H 4775 4475 50  0001 C CNN
 	1    4775 4475
@@
 F 0 "C92" H 5350 4975 50  0000 L CNN
 F 1 "1nF" H 5175 4800 50  0000 L CNN
-F 2 "Atari:C_Axial_L5.1mm_D2.5mm_P12.50mm_Horizontal" H 5363 4750 50  0001 C CNN
+F 2 "Capacitor_SMD:C_1206_3216Metric_Pad1.42x1.75mm_HandSolder" H 5363 4750 50  0001 C CNN
 F 3 "~" H 5325 4900 50  0001 C CNN
 	1    5325 4900
@@
 F 0 "C91" H 5600 4975 50  0000 L CNN
 F 1 "1nF" H 5425 4800 50  0000 L CNN
-F 2 "Atari:C_Axial_L5.1mm_D2.5mm_P12.50mm_Horizontal" H 5613 4750 50  0001 C CNN
+F 2 "Capacitor_SMD:C_1206_3216Metric_Pad1.42x1.75mm_HandSolder" H 5613 4750 50  0001 C CNN
 F 3 "~" H 5575 4900 50  0001 C CNN
 	1    5575 4900
@@
 F 0 "C90" H 5850 4975 50  0000 L CNN
 F 1 "1nF" H 5675 4800 50  0000 L CNN
-F 2 "Atari:C_Axial_L5.1mm_D2.5mm_P12.50mm_Horizontal" H 5863 4750 50  0001 C CNN
+F 2 "Capacitor_SMD:C_1206_3216Metric_Pad1.42x1.75mm_HandSolder" H 5863 4750 50  0001 C CNN
 F 3 "~" H 5825 4900 50  0001 C CNN
 	1    5825 4900
@@
 F 0 "C89" H 6100 4975 50  0000 L CNN
 F 1 "1nF" H 5925 4800 50  0000 L CNN
-F 2 "Atari:C_Axial_L5.1mm_D2.5mm_P12.50mm_Horizontal" H 6113 4750 50  0001 C CNN
+F 2 "Capacitor_SMD:C_1206_3216Metric_Pad1.42x1.75mm_HandSolder" H 6113 4750 50  0001 C CNN
 F 3 "~" H 6075 4900 50  0001 C CNN
 	1    6075 4900
@@
 F 0 "C88" H 6350 4975 50  0000 L CNN
 F 1 "1nF" H 6175 4800 50  0000 L CNN
-F 2 "Atari:C_Axial_L5.1mm_D2.5mm_P12.50mm_Horizontal" H 6363 4750 50  0001 C CNN
+F 2 "Capacitor_SMD:C_1206_3216Metric_Pad1.42x1.75mm_HandSolder" H 6363 4750 50  0001 C CNN
 F 3 "~" H 6325 4900 50  0001 C CNN
 	1    6325 4900
@@
 F 0 "C87" H 6600 4975 50  0000 L CNN
 F 1 "1nF" H 6425 4800 50  0000 L CNN
-F 2 "Atari:C_Axial_L5.1mm_D2.5mm_P12.50mm_Horizontal" H 6613 4750 50  0001 C CNN
+F 2 "Capacitor_SMD:C_1206_3216Metric_Pad1.42x1.75mm_HandSolder" H 6613 4750 50  0001 C CNN
 F 3 "~" H 6575 4900 50  0001 C CNN
 	1    6575 4900
@@
 F 0 "C86" H 6850 4975 50  0000 L CNN
 F 1 "1nF" H 6675 4800 50  0000 L CNN
-F 2 "Atari:C_Axial_L5.1mm_D2.5mm_P12.50mm_Horizontal" H 6863 4750 50  0001 C CNN
+F 2 "Capacitor_SMD:C_1206_3216Metric_Pad1.42x1.75mm_HandSolder" H 6863 4750 50  0001 C CNN
 F 3 "~" H 6825 4900 50  0001 C CNN
 	1    6825 4900
@@
 F 0 "C85" H 7100 4975 50  0000 L CNN
 F 1 "1nF" H 6925 4800 50  0000 L CNN
-F 2 "Atari:C_Axial_L5.1mm_D2.5mm_P12.50mm_Horizontal" H 7113 4750 50  0001 C CNN
+F 2 "Capacitor_SMD:C_1206_3216Metric_Pad1.42x1.75mm_HandSolder" H 7113 4750 50  0001 C CNN
 F 3 "~" H 7075 4900 50  0001 C CNN
 	1    7075 4900
@@
 F 0 "L29" V 7650 3600 50  0000 C CNN
 F 1 "10uH" V 7550 3775 50  0000 C CNN
-F 2 "Atari:L_Axial_L7.0mm_D3.3mm_P12.50mm_Horizontal_Fastron_MICC" H 7600 3775 50  0001 C CNN
+F 2 "Inductor_SMD:L_1812_4532Metric_Pad1.30x3.40mm_HandSolder" H 7600 3775 50  0001 C CNN
 F 3 "~" H 7600 3775 50  0001 C CNN
 	1    7600 3775
@@
 F 0 "L28" V 7650 3700 50  0000 C CNN
 F 1 "10uH" V 7575 3900 50  0000 C CNN
-F 2 "Atari:L_Axial_L7.0mm_D3.3mm_P12.50mm_Horizontal_Fastron_MICC" H 7600 3875 50  0001 C CNN
+F 2 "Inductor_SMD:L_1812_4532Metric_Pad1.30x3.40mm_HandSolder" H 7600 3875 50  0001 C CNN
 F 3 "~" H 7600 3875 50  0001 C CNN
 	1    7600 3875
@@
 F 0 "L27" V 7650 3800 50  0000 C CNN
 F 1 "10uH" V 7575 4000 50  0000 C CNN
-F 2 "Atari:L_Axial_L7.0mm_D3.3mm_P12.50mm_Horizontal_Fastron_MICC" H 7600 3975 50  0001 C CNN
+F 2 "Inductor_SMD:L_1812_4532Metric_Pad1.30x3.40mm_HandSolder" H 7600 3975 50  0001 C CNN
 F 3 "~" H 7600 3975 50  0001 C CNN
 	1    7600 3975
@@
 F 0 "L26" V 7650 3900 50  0000 C CNN
 F 1 "10uH" V 7575 4100 50  0000 C CNN
-F 2 "Atari:L_Axial_L7.0mm_D3.3mm_P12.50mm_Horizontal_Fastron_MICC" H 7600 4075 50  0001 C CNN
+F 2 "Inductor_SMD:L_1812_4532Metric_Pad1.30x3.40mm_HandSolder" H 7600 4075 50  0001 C CNN
 F 3 "~" H 7600 4075 50  0001 C CNN
 	1    7600 4075
@@
 F 0 "L22" V 7650 4000 50  0000 C CNN
 F 1 "10uH" V 7575 4200 50  0000 C CNN
-F 2 "Atari:L_Axial_L7.0mm_D3.3mm_P12.50mm_Horizontal_Fastron_MICC" H 7600 4175 50  0001 C CNN
+F 2 "Inductor_SMD:L_1812_4532Metric_Pad1.30x3.40mm_HandSolder" H 7600 4175 50  0001 C CNN
 F 3 "~" H 7600 4175 50  0001 C CNN
 	1    7600 4175
@@
 F 0 "L21" V 7650 4100 50  0000 C CNN
 F 1 "10uH" V 7575 4300 50  0000 C CNN
-F 2 "Atari:L_Axial_L7.0mm_D3.3mm_P12.50mm_Horizontal_Fastron_MICC" H 7600 4275 50  0001 C CNN
+F 2 "Inductor_SMD:L_1812_4532Metric_Pad1.30x3.40mm_HandSolder" H 7600 4275 50  0001 C CNN
 F 3 "~" H 7600 4275 50  0001 C CNN
 	1    7600 4275
@@
 F 0 "L20" V 7650 4200 50  0000 C CNN
 F 1 "10uH" V 7575 4400 50  0000 C CNN
-F 2 "Atari:L_Axial_L7.0mm_D3.3mm_P12.50mm_Horizontal_Fastron_MICC" H 7600 4375 50  0001 C CNN
+F 2 "Inductor_SMD:L_1812_4532Metric_Pad1.30x3.40mm_HandSolder" H 7600 4375 50  0001 C CNN
 F 3 "~" H 7600 4375 50  0001 C CNN
 	1    7600 4375
@@
 F 0 "L19" V 7650 4300 50  0000 C CNN
 F 1 "10uH" V 7575 4500 50  0000 C CNN
-F 2 "Atari:L_Axial_L7.0mm_D3.3mm_P12.50mm_Horizontal_Fastron_MICC" H 7600 4475 50  0001 C CNN
+F 2 "Inductor_SMD:L_1812_4532Metric_Pad1.30x3.40mm_HandSolder" H 7600 4475 50  0001 C CNN
 F 3 "~" H 7600 4475 50  0001 C CNN
 	1    7600 4475

Commit message: OSS and Basic in PLCC
Parts:
- C68: footprint Atari:C_Axial_L5.1mm_D2.5mm_P12.50mm_Horizontal -> Capacitor_SMD:C_1206_3216Metric_Pad1.42x1.75mm_HandSolder
- R23, R24, R25, R501, R85, R86, R87, R88: footprint Atari:R_Axial_DIN0207_L3.6mm_D2.2mm_P10.16mm_Horizontal -> Resistor_SMD:R_1206_3216Metric_Pad1.42x1.75mm_HandSolder
Changed lines of the file:
@@
 F 0 "R88" V 1725 2350 50  0000 L CNN
 F 1 "3k" H 1625 2575 50  0000 L CNN
-F 2 "Atari:R_Axial_DIN0207_L3.6mm_D2.2mm_P10.16mm_Horizontal" V 1655 2425 50  0001 C CNN
+F 2 "Resistor_SMD:R_1206_3216Metric_Pad1.42x1.75mm_HandSolder" V 1655 2425 50  0001 C CNN
 F 3 "~" H 1725 2425 50  0001 C CNN
 	1    1725 2425
@@
 F 0 "R85" V 1900 2350 50  0000 L CNN
 F 1 "3k" H 1800 2575 50  0000 L CNN
-F 2 "Atari:R_Axial_DIN0207_L3.6mm_D2.2mm_P10.16mm_Horizontal" V 1830 2425 50  0001 C CNN
+F 2 "Resistor_SMD:R_1206_3216Metric_Pad1.42x1.75mm_HandSolder" V 1830 2425 50  0001 C CNN
 F 3 "~" H 1900 2425 50  0001 C CNN
 	1    1900 2425
@@
 F 0 "R25" V 2075 2350 50  0000 L CNN
 F 1 "3k" H 1975 2575 50  0000 L CNN
-F 2 "Atari:R_Axial_DIN0207_L3.6mm_D2.2mm_P10.16mm_Horizontal" V 2005 2425 50  0001 C CNN
+F 2 "Resistor_SMD:R_1206_3216Metric_Pad1.42x1.75mm_HandSolder" V 2005 2425 50  0001 C CNN
 F 3 "~" H 2075 2425 50  0001 C CNN
 	1    2075 2425
@@
 F 0 "R23" V 2250 2350 50  0000 L CNN
 F 1 "3k" H 2150 2575 50  0000 L CNN
-F 2 "Atari:R_Axial_DIN0207_L3.6mm_D2.2mm_P10.16mm_Horizontal" V 2180 2425 50  0001 C CNN
+F 2 "Resistor_SMD:R_1206_3216Metric_Pad1.42x1.75mm_HandSolder" V 2180 2425 50  0001 C CNN
 F 3 "~" H 2250 2425 50  0001 C CNN
 	1    2250 2425
@@
 F 0 "R24" V 2425 2350 50  0000 L CNN
 F 1 "3k" H 2325 2575 50  0000 L CNN
-F 2 "Atari:R_Axial_DIN0207_L3.6mm_D2.2mm_P10.16mm_Horizontal" V 2355 2425 50  0001 C CNN
+F 2 "Resistor_SMD:R_1206_3216Metric_Pad1.42x1.75mm_HandSolder" V 2355 2425 50  0001 C CNN
 F 3 "~" H 2425 2425 50  0001 C CNN
 	1    2425 2425
@@
 F 0 "R87" V 2950 2350 50  0000 L CNN
 F 1 "3k" H 2850 2575 50  0000 L CNN
-F 2 "Atari:R_Axial_DIN0207_L3.6mm_D2.2mm_P10.16mm_Horizontal" V 2880 2425 50  0001 C CNN
+F 2 "Resistor_SMD:R_1206_3216Metric_Pad1.42x1.75mm_HandSolder" V 2880 2425 50  0001 C CNN
 F 3 "~" H 2950 2425 50  0001 C CNN
 	1    2950 2425
@@
 F 0 "R86" V 2375 3800 50  0000 L CNN
 F 1 "3k" H 2275 4025 50  0000 L CNN
-F 2 "Atari:R_Axial_DIN0207_L3.6mm_D2.2mm_P10.16mm_Horizontal" V 2305 3875 50  0001 C CNN
+F 2 "Resistor_SMD:R_1206_3216Metric_Pad1.42x1.75mm_HandSolder" V 2305 3875 50  0001 C CNN
 F 3 "~" H 2375 3875 50  0001 C CNN
 	1    2375 3875
@@
 F 0 "C68" H 2915 5871 50  0000 L CNN
 F 1 "100nF" H 2915 5780 50  0000 L CNN
-F 2 "Atari:C_Axial_L5.1mm_D2.5mm_P12.50mm_Horizontal" H 2838 5675 50  0001 C CNN
+F 2 "Capacitor_SMD:C_1206_3216Metric_Pad1.42x1.75mm_HandSolder" H 2838 5675 50  0001 C CNN
 F 3 "~" H 2800 5825 50  0001 C CNN
 	1    2800 5825
@@
 F 0 "R501" V 2775 2325 50  0000 L CNN
 F 1 "3k" H 2675 2575 50  0000 L CNN
-F 2 "Atari:R_Axial_DIN0207_L3.6mm_D2.2mm_P10.16mm_Horizontal" V 2705 2425 50  0001 C CNN
+F 2 "Resistor_SMD:R_1206_3216Metric_Pad1.42x1.75mm_HandSolder" V 2705 2425 50  0001 C CNN
 F 3 "~" H 2775 2425 50  0001 C CNN
 	1    2775 2425

Commit message: Final modification
Parts:
- C79: footprint Capacitor_THT:CP_Axial_L11.0mm_D5.0mm_P18.00mm_Horizontal -> Capacitor_THT:CP_Radial_D7.5mm_P2.50mm
- C80: footprint Atari:C_Axial_L5.1mm_D2.5mm_P12.50mm_Horizontal -> Resistor_SMD:R_1206_3216Metric_Pad1.42x1.75mm_HandSolder
- C81, C82, C83, C84: footprint Atari:C_Axial_L5.1mm_D2.5mm_P12.50mm_Horizontal -> Capacitor_SMD:C_1206_3216Metric_Pad1.42x1.75mm_HandSolder
- FB10, FB11: footprint Atari:L_Axial_L7.0mm_D3.3mm_P12.50mm_Horizontal_Fastron_MICC -> Inductor_SMD:L_1812_4532Metric_Pad1.30x3.40mm_HandSolder
- R117, R118, R119, R91, R92, R93, R94: footprint Atari:R_Axial_DIN0207_L3.6mm_D2.2mm_P10.16mm_Horizontal -> Resistor_SMD:R_1206_3216Metric_Pad1.42x1.75mm_HandSolder
Changed lines of the file:
@@
 F 0 "R91" V 4725 2450 50  0000 L CNN
 F 1 "2k7" H 4575 2675 50  0000 L CNN
-F 2 "Atari:R_Axial_DIN0207_L3.6mm_D2.2mm_P10.16mm_Horizontal" V 4655 2525 50  0001 C CNN
+F 2 "Resistor_SMD:R_1206_3216Metric_Pad1.42x1.75mm_HandSolder" V 4655 2525 50  0001 C CNN
 F 3 "~" H 4725 2525 50  0001 C CNN
 	1    4725 2525
@@
 F 0 "FB11" V 5801 1850 50  0000 C CNN
 F 1 "Ferrite_Bead" V 5892 1850 50  0000 C CNN
-F 2 "Atari:L_Axial_L7.0mm_D3.3mm_P12.50mm_Horizontal_Fastron_MICC" V 6005 1850 50  0001 C CNN
+F 2 "Inductor_SMD:L_1812_4532Metric_Pad1.30x3.40mm_HandSolder" V 6005 1850 50  0001 C CNN
 F 3 "~" H 6075 1850 50  0001 C CNN
 	1    6075 1850
@@
 F 0 "FB10" V 6000 2525 50  0000 C CNN
 F 1 "Ferrite_Bead" V 6175 2350 50  0000 C CNN
-F 2 "Atari:L_Axial_L7.0mm_D3.3mm_P12.50mm_Horizontal_Fastron_MICC" V 6005 2350 50  0001 C CNN
+F 2 "Inductor_SMD:L_1812_4532Metric_Pad1.30x3.40mm_HandSolder" V 6005 2350 50  0001 C CNN
 F 3 "~" H 6075 2350 50  0001 C CNN
 	1    6075 2350
@@
 F 0 "C79" H 7218 2446 50  0000 L CNN
 F 1 "22uF" H 7218 2355 50  0000 L CNN
-F 2 "Capacitor_THT:CP_Axial_L11.0mm_D5.0mm_P18.00mm_Horizontal" H 7138 2250 50  0001 C CNN
+F 2 "Capacitor_THT:CP_Radial_D7.5mm_P2.50mm" H 7138 2250 50  0001 C CNN
 F 3 "~" H 7100 2400 50  0001 C CNN
 	1    7100 2400
@@
 F 0 "C80" H 7550 2475 50  0000 L CNN
 F 1 "1nF" H 7375 2300 50  0000 L CNN
-F 2 "Atari:C_Axial_L5.1mm_D2.5mm_P12.50mm_Horizontal" H 7563 2250 50  0001 C CNN
+F 2 "Resistor_SMD:R_1206_3216Metric_Pad1.42x1.75mm_HandSolder" H 7563 2250 50  0001 C CNN
 F 3 "~" H 7525 2400 50  0001 C CNN
 	1    7525 2400
@@
 F 0 "C81" H 7925 2475 50  0000 L CNN
 F 1 "1nF" H 7750 2300 50  0000 L CNN
-F 2 "Atari:C_Axial_L5.1mm_D2.5mm_P12.50mm_Horizontal" H 7938 2250 50  0001 C CNN
+F 2 "Capacitor_SMD:C_1206_3216Metric_Pad1.42x1.75mm_HandSolder" H 7938 2250 50  0001 C CNN
 F 3 "~" H 7900 2400 50  0001 C CNN
 	1    7900 2400
@@
 F 0 "R92" V 5275 2875 50  0000 L CNN
 F 1 "4k7" V 5200 2700 50  0000 L CNN
-F 2 "Atari:R_Axial_DIN0207_L3.6mm_D2.2mm_P10.16mm_Horizontal" V 5205 2950 50  0001 C CNN
+F 2 "Resistor_SMD:R_1206_3216Metric_Pad1.42x1.75mm_HandSolder" V 5205 2950 50  0001 C CNN
 F 3 "~" H 5275 2950 50  0001 C CNN
 	1    5275 2950
@@
 F 0 "R94" V 5825 2875 50  0000 L CNN
 F 1 "4k7" V 5750 2700 50  0000 L CNN
-F 2 "Atari:R_Axial_DIN0207_L3.6mm_D2.2mm_P10.16mm_Horizontal" V 5755 2950 50  0001 C CNN
+F 2 "Resistor_SMD:R_1206_3216Metric_Pad1.42x1.75mm_HandSolder" V 5755 2950 50  0001 C CNN
 F 3 "~" H 5825 2950 50  0001 C CNN
 	1    5825 2950
@@
 F 0 "R117" V 6600 3225 50  0000 L CNN
 F 1 "100" V 6550 3450 50  0000 L CNN
-F 2 "Atari:R_Axial_DIN0207_L3.6mm_D2.2mm_P10.16mm_Horizontal" V 6530 3325 50  0001 C CNN
+F 2 "Resistor_SMD:R_1206_3216Metric_Pad1.42x1.75mm_HandSolder" V 6530 3325 50  0001 C CNN
 F 3 "~" H 6600 3325 50  0001 C CNN
 	1    6600 3325
@@
 F 0 "R118" V 6600 3325 50  0000 L CNN
 F 1 "220" V 6550 3550 50  0000 L CNN
-F 2 "Atari:R_Axial_DIN0207_L3.6mm_D2.2mm_P10.16mm_Horizontal" V 6530 3425 50  0001 C CNN
+F 2 "Resistor_SMD:R_1206_3216Metric_Pad1.42x1.75mm_HandSolder" V 6530 3425 50  0001 C CNN
 F 3 "~" H 6600 3425 50  0001 C CNN
 	1    6600 3425
@@
 F 0 "R119" V 6600 3425 50  0000 L CNN
 F 1 "100" V 6550 3650 50  0000 L CNN
-F 2 "Atari:R_Axial_DIN0207_L3.6mm_D2.2mm_P10.16mm_Horizontal" V 6530 3525 50  0001 C CNN
+F 2 "Resistor_SMD:R_1206_3216Metric_Pad1.42x1.75mm_HandSolder" V 6530 3525 50  0001 C CNN
 F 3 "~" H 6600 3525 50  0001 C CNN
 	1    6600 3525
@@
 F 0 "R93" V 6600 2600 50  0000 L CNN
 F 1 "4k7" V 6550 2825 50  0000 L CNN
-F 2 "Atari:R_Axial_DIN0207_L3.6mm_D2.2mm_P10.16mm_Horizontal" V 6530 2700 50  0001 C CNN
+F 2 "Resistor_SMD:R_1206_3216Metric_Pad1.42x1.75mm_HandSolder" V 6530 2700 50  0001 C CNN
 F 3 "~" H 6600 2700 50  0001 C CNN
 	1    6600 2700
@@
 F 0 "C84" H 8700 5000 50  0000 L CNN
 F 1 "1nF" H 8525 4825 50  0000 L CNN
-F 2 "Atari:C_Axial_L5.1mm_D2.5mm_P12.50mm_Horizontal" H 8713 4775 50  0001 C CNN
+F 2 "Capacitor_SMD:C_1206_3216Metric_Pad1.42x1.75mm_HandSolder" H 8713 4775 50  0001 C CNN
 F 3 "~" H 8675 4925 50  0001 C CNN
 	1    8675 4925
@@
 F 0 "C83" H 9050 5000 50  0000 L CNN
 F 1 "1nF" H 8875 4825 50  0000 L CNN
-F 2 "Atari:C_Axial_L5.1mm_D2.5mm_P12.50mm_Horizontal" H 9063 4775 50  0001 C CNN
+F 2 "Capacitor_SMD:C_1206_3216Metric_Pad1.42x1.75mm_HandSolder" H 9063 4775 50  0001 C CNN
 F 3 "~" H 9025 4925 50  0001 C CNN
 	1    9025 4925
@@
 F 0 "C82" H 9400 5000 50  0000 L CNN
 F 1 "1nF" H 9225 4825 50  0000 L CNN
-F 2 "Atari:C_Axial_L5.1mm_D2.5mm_P12.50mm_Horizontal" H 9413 4775 50  0001 C CNN
+F 2 "Capacitor_SMD:C_1206_3216Metric_Pad1.42x1.75mm_HandSolder" H 9413 4775 50  0001 C CNN
 F 3 "~" H 9375 4925 50  0001 C CNN
 	1    9375 4925
