File: Power.sch (KiCad schematic (older format))
At the start: 22 parts, among them J7 Power, SW1 Switch_power_on

Commit message: Final modification
Parts:
- added J11, J12, J13, J14, J15, J16, J17, J18, J19, J20, J21: C, Connector_PinHeader_2.54mm:PinHeader_1x01_P2.54mm_Vertical, symbol Connector_Generic:Conn_01x01
- C10, C2, C3: footprint Capacitor_THT:CP_Axial_L11.0mm_D5.0mm_P18.00mm_Horizontal -> Capacitor_THT:CP_Radial_D7.5mm_P2.50mm
Connections:
- net +5VA: now also J18.1 (Pin_1), J19.1 (Pin_1)
- net GND: now also J14.1 (Pin_1), J15.1 (Pin_1), J16.1 (Pin_1), J17.1 (Pin_1), J20.1 (Pin_1), J21.1 (Pin_1)
- net at C1.1, C2.1, C3.1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: now also J12.1 (Pin_1), J13.1 (Pin_1)
